Commit message: tidying up

File: catkin_ws/src/my_robot/urdf/my_robot.xacro (robot description, xacro)
@@ -22,5 +22,5 @@
       <origin xyz="0 0 0" rpy=" 0 0 0"/>
       <geometry>
-        <box size=".4 .2 .1"/>
+        <box size=".5 .2 .1"/>
       </geometry>
     </collision>
@@ -28,11 +28,25 @@
       <origin xyz="0 0 0" rpy=" 0 0 0"/>
       <geometry>
-        <box size=".4 .2 .1"/>
+        <box size=".5 .2 .1"/>
       </geometry>
+        <material name="chassis_material">
+          <lighting>1</lighting>
+          <script>
+            <uri>file://media/materials/scripts/gazebo.material</uri>
+            <name>Gazebo/GreenGlow</name>
+          </script>
+          <ambient>0.3 0.3 0.3 1</ambient>
+          <diffuse>0.7 0.7 0.7 1</diffuse>
+          <specular>0.01 0.01 0.01 1</specular>
+          <emissive>0 0 0 1</emissive>
+          <shader type='vertex'>
+            <normal_map>__default__</normal_map>
+          </shader>
+        </material>
     </visual>
     <collision name='back_caster_collision'>
       <origin xyz="-0.15 0 -0.05" rpy=" 0 0 0"/>
       <geometry>
-        <sphere radius="0.0499"/>
+        <sphere radius="0.0999"/>
       </geometry>
     </collision>
@@ -40,5 +54,5 @@
       <origin xyz="-0.15 0 -0.05" rpy=" 0 0 0"/>
       <geometry>
-        <sphere radius="0.05"/>
+        <sphere radius="0.10"/>
       </geometry>
     </visual>
@@ -46,5 +60,5 @@
       <origin xyz="0.15 0 -0.05" rpy=" 0 0 0"/>
       <geometry>
-        <sphere radius="0.0499"/>
+        <sphere radius="0.0999"/>
       </geometry>
     </collision>
@@ -52,5 +66,5 @@
       <origin xyz="0.15 0 -0.05" rpy=" 0 0 0"/>
       <geometry>
-        <sphere radius="0.05"/>
+        <sphere radius="0.10"/>
       </geometry>
     </visual>
@@ -69,5 +83,5 @@
 			<origin xyz="0.0 0 0" rpy=" 0 1.5707 1.5707"/>
 			<geometry>
-				<cylinder radius="0.1" length="0.05"/>
+				<cylinder radius="0.15" length="0.05"/>
 			</geometry>
 		</collision>
@@ -75,5 +89,5 @@
 			<origin xyz="0.0 0 0" rpy=" 0 1.5707 1.5707"/>
 			<geometry>
-				<cylinder radius="0.1" length="0.05"/>
+				<cylinder radius="0.15" length="0.05"/>
 			</geometry>
 		</visual>
@@ -92,5 +106,5 @@
 			<origin xyz="0.0 -.15 0" rpy=" 0 1.5707 1.5707"/>
 			<geometry>
-				<cylinder radius="0.1" length="0.05"/>
+				<cylinder radius="0.15" length="0.05"/>
 			</geometry>
 		</collision>
@@ -98,5 +112,5 @@
 			<origin xyz="0.0 -.15 0" rpy=" 0 1.5707 1.5707"/>
 			<geometry>
-				<cylinder radius="0.1" length="0.05"/>
+				<cylinder radius="0.15" length="0.05"/>
 			</geometry>
 		</visual>
@@ -140,5 +154,5 @@
 	</link>
 	<joint type='continuous' name='camera_joint'>
-		<origin xyz="0.2 0 0" rpy="0 0 0"/>
+		<origin xyz="0.25 0 0" rpy="0 0 0"/>
 		<child link='camera'/>
 		<parent link='chassis'/>
